Commit message: Simulated in gazebo

File: description/urdf/ack.urdf.xacro (robot description, xacro)
@@ -1,199 +1,6 @@
-<?xml version="1.0" encoding="utf-8"?>
-<robot name="ackerman_simple">
-  <xacro:include filename="$(find description)/urdf/gazebo.xacro"/>
-  <xacro:include filename="$(find description)/urdf/ros2_control.xacro"/>
-  <!-- ================= BASE ================= -->
-  <link name="base_footprint"/>
-  <link name="base_link">
-    <inertial>
-      <origin xyz="0.0115 0 0.0687" rpy="0 0 0" />
-      <mass value="1.8886" />
-      <inertia ixx="0.00576" ixy="0.0" ixz="0.000003" iyy="0.01878" iyz="0.0" izz="0.02437" />
-    </inertial>
-    <!-- Chassis Box -->
-    <visual>
-      <origin xyz="0.01 0 0.05" rpy="0 0 0" />
-      <geometry>
-        <box size="0.35 0.15 0.08"/>
-      </geometry>
-      <material name="blue">
-        <color rgba="0.2 0.2 0.8 1" />
-      </material>
-    </visual>
-    <collision>
-      <origin xyz="0.01 0 0.05" rpy="0 0 0" />
-      <geometry>
-        <box size="0.35 0.15 0.08"/>
-      </geometry>
-    </collision>
-  </link>
-  <joint name="base_joint" type="fixed">
-    <origin xyz="-0.0117 0 0.02677" rpy="0 0 0" />
-    <parent link="base_footprint" />
-    <child link="base_link" />
-  </joint>
-  <!-- ================= FRONT LEFT STEERING & WHEEL ================= -->
-  <link name="FL_STEERING_LINK">
-    <inertial>
-      <origin xyz="-0.0029 0 0" rpy="0 0 0" />
-      <mass value="0.0038" />
-      <inertia ixx="0.0000003" ixy="0" ixz="0" iyy="0.0000006" iyz="0" izz="0.0000003" />
-    </inertial>
-  </link>
-  <joint name="FL_STEERING_JOINT" type="revolute">
-    <origin xyz="0.16174 0.085 0.0235" rpy="0 0 0" />
-    <parent link="base_link" />
-    <child link="FL_STEERING_LINK" />
-    <axis xyz="0 0 1" />
-    <limit lower="-0.524" upper="0.524" effort="5" velocity="3" />
-  </joint>
-  <link name="FL_WHEEL_LINK">
-    <inertial>
-      <origin xyz="0 0 0" rpy="0 0 0" />
-      <mass value="0.0635" />
-      <inertia ixx="0.000046" ixy="0" ixz="0" iyy="0.000089" iyz="0" izz="0.000046" />
-    </inertial>
-    <visual>
-      <origin xyz="0 0 0" rpy="1.57079632679 0 0" />
-      <geometry>
-        <cylinder radius="0.05027" length="0.03"/>
-      </geometry>
-      <material name="black"><color rgba="0.1 0.1 0.1 1"/></material>
-    </visual>
-    <collision>
-      <origin xyz="0 0 0" rpy="1.57079632679 0 0" />
-      <geometry>
-        <cylinder radius="0.05027" length="0.03"/>
-      </geometry>
-    </collision>
-  </link>
-  <joint name="FL_WHEEL_JOINT" type="continuous">
-    <origin xyz="0 0.0245 0" rpy="0 0 0" />
-    <parent link="FL_STEERING_LINK" />
-    <child link="FL_WHEEL_LINK" />
-    <axis xyz="0 1 0" />
-  </joint>
-  <!-- ================= FRONT RIGHT STEERING & WHEEL ================= -->
-  <link name="FR_STEERING_LINK">
-    <inertial>
-      <origin xyz="0.0015 0 0" rpy="0 0 0" />
-      <mass value="0.0047" />
-      <inertia ixx="0.0000003" ixy="0" ixz="0" iyy="0.000001" iyz="0" izz="0.0000007" />
-    </inertial>
-  </link>
-  <joint name="FR_STEERING_JOINT" type="revolute">
-    <origin xyz="0.16174 -0.085 0.0235" rpy="0 0 0" />
-    <parent link="base_link" />
-    <child link="FR_STEERING_LINK" />
-    <axis xyz="0 0 1" />
-    <limit lower="-0.524" upper="0.524" effort="5" velocity="3" />
-    <mimic joint="FL_STEERING_JOINT" multiplier="1.0" offset="0.0" />
-  </joint>
-  <link name="FR_WHEEL_LINK">
-    <inertial>
-      <origin xyz="0 0 0" rpy="0 0 0" />
-      <mass value="0.0635" />
-      <inertia ixx="0.000046" ixy="0" ixz="0" iyy="0.000089" iyz="0" izz="0.000046" />
-    </inertial>
-    <visual>
-      <origin xyz="0 0 0" rpy="1.57079632679 0 0" />
-      <geometry>
-        <cylinder radius="0.05027" length="0.03"/>
-      </geometry>
-      <material name="black"><color rgba="0.1 0.1 0.1 1"/></material>
-    </visual>
-    <collision>
-      <origin xyz="0 0 0" rpy="1.57079632679 0 0" />
-      <geometry>
-        <cylinder radius="0.05027" length="0.03"/>
-      </geometry>
-    </collision>
-  </link>
-  <joint name="FR_WHEEL_JOINT" type="continuous">
-    <origin xyz="0 -0.0245 0" rpy="0 0 0" />
-    <parent link="FR_STEERING_LINK" />
-    <child link="FR_WHEEL_LINK" />
-    <axis xyz="0 1 0" />
-  </joint>
-  <!-- ================= REAR LEFT WHEEL ================= -->
-  <link name="BL_WHEEL_LINK">
-    <inertial>
-      <origin xyz="0 0 0" rpy="0 0 0" />
-      <mass value="0.0616" />
-      <inertia ixx="0.000046" ixy="0" ixz="0" iyy="0.000089" iyz="0" izz="0.000046" />
-    </inertial>
-    <visual>
-      <origin xyz="0 0 0" rpy="1.57079632679 0 0" />
-      <geometry>
-        <cylinder radius="0.05027" length="0.03"/>
-      </geometry>
-      <material name="black"><color rgba="0.1 0.1 0.1 1"/></material>
-    </visual>
-    <collision>
-      <origin xyz="0 0 0" rpy="1.57079632679 0 0" />
-      <geometry>
-        <cylinder radius="0.05027" length="0.03"/>
-      </geometry>
-    </collision>
-  </link>
-  <joint name="BL_WHEEL_JOINT" type="continuous">
-    <!-- Reverted Z back to 0.02075 -->
-    <origin xyz="-0.13328 0.1093 0.02075" rpy="0 0 0" />
-    <parent link="base_link" />
-    <child link="BL_WHEEL_LINK" />
-    <axis xyz="0 1 0" />
-  </joint>
-  <!-- ================= REAR RIGHT WHEEL ================= -->
-  <link name="BR_WHEEL_LINK">
-    <inertial>
-      <origin xyz="0 0 0" rpy="0 0 0" />
-      <mass value="0.0616" />
-      <inertia ixx="0.000046" ixy="0" ixz="0" iyy="0.000089" iyz="0" izz="0.000046" />
-    </inertial>
-    <visual>
-      <origin xyz="0 0 0" rpy="1.57079632679 0 0" />
-      <geometry>
-        <cylinder radius="0.05027" length="0.03"/>
-      </geometry>
-      <material name="black"><color rgba="0.1 0.1 0.1 1"/></material>
-    </visual>
-    <collision>
-      <origin xyz="0 0 0" rpy="1.57079632679 0 0" />
-      <geometry>
-        <cylinder radius="0.05027" length="0.03"/>
-      </geometry>
-    </collision>
-  </link>
-  <joint name="BR_WHEEL_JOINT" type="continuous">
-    <!-- Reverted Z back to 0.02075 -->
-    <origin xyz="-0.13328 -0.1093 0.02075" rpy="0 0 0" />
-    <parent link="base_link" />
-    <child link="BR_WHEEL_LINK" />
-    <axis xyz="0 1 0" />
-  </joint>
-    <!-- ================= CAMERA ================= -->
-  <link name="CAMERA_LINK">
-    <inertial>
-      <origin xyz="0 0 0" rpy="0 0 0" />
-      <mass value="0.0548" />
-      <inertia ixx="0.000069" ixy="0" ixz="0" iyy="0.000004" iyz="0" izz="0.000066" />
-    </inertial>
-    <visual>
-      <origin xyz="0 0 0" rpy="0 0 0" />
-      <geometry>
-        <box size="0.02 0.06 0.02"/>
-      </geometry>
-      <material name="red"><color rgba="0.8 0.1 0.1 1"/></material>
-    </visual>
-    <collision>
-      <origin xyz="0 0 0" rpy="0 0 0" />
-      <geometry>
-        <box size="0.02 0.06 0.02"/>
-      </geometry>
-    </collision>
-  </link>
-  <joint name="CAMERA_JOINT" type="fixed">
-    <origin xyz="0.15 0.0 0.2" rpy="0 0.1 0" />
-    <parent link="base_link" />
-    <child link="CAMERA_LINK" />
-  </joint>
+<?xml version="1.0" ?>
+<robot name="ackerman_simple" xmlns:xacro="http://www.ros.org/wiki/xacro">
+    <xacro:include filename="$(find description)/urdf/gazebo.xacro" />
+    <xacro:include filename="$(find description)/urdf/ros2_control.xacro" />
+    <xacro:include filename="$(find description)/urdf/ack.xacro" />
+</robot>
