Commit message: Camera Image spawned

File: description/urdf/gazebo.xacro (robot description, xacro)
@@ -1,24 +1,31 @@
 <?xml version="1.0"?>
 <robot xmlns:xacro="http://www.ros.org/wiki/xacro">
-  <gazebo reference="CAMERA_LINK">
-    <sensor name="camera_sensor" type="camera">
-      <always_on>true</always_on>
-      <visualize>true</visualize>
-      <update_rate>30</update_rate>
-      <topic>camera/image_raw</topic>
-      <gz_frame_id>CAMERA_LINK</gz_frame_id>
-      <camera>
-        <horizontal_fov>1.047</horizontal_fov>
-        <image>
-          <width>640</width>
-          <height>480</height>
-          <format>R8G8B8</format>
-        </image>
-        <clip>
-          <near>0.05</near>
-          <far>20.0</far>
-        </clip>
-      </camera>
-    </sensor>
-  </gazebo>
+    <gazebo reference="CAMERA_LINK">
+        <material>Gazebo/Green</material>
+        <sensor name="camera" type="camera">
+          <pose> 0 0 0 0 0 0</pose>
+          <visualize>true</visualize>
+          <update_rate>10</update_rate>
+          <camera>
+            <camera_info_topic>camera/camera_info</camera_info_topic>
+            <horizontal_fov>1.089</horizontal_fov>
+              <image>
+                <format>R8G8B8</format>
+                <width>640</width>
+                <height>480</height>
+              </image>
+              <clip>
+                <near>0.05</near>
+                <far>8.0</far>
+              </clip>
+          </camera>
+          <topic>camera/image_raw</topic>
+          <gz_frame_id>camera_link_optical</gz_frame_id>
+        </sensor>
+    </gazebo>
+    <gazebo>
+      <plugin filename="ignition-gazebo-sensors-system" name="ignition::gazebo::systems::Sensors">
+        <render_engine>ogre2</render_engine>
+      </plugin>
+    </gazebo>
 </robot>
