Commit message: Vision node

File: description/urdf/ack.xacro (robot description, xacro)
@@ -196,3 +196,9 @@
     <child link="CAMERA_LINK" />
   </joint>
+  <joint name="camera_optical_joint" type="fixed">
+        <parent link="CAMERA_LINK"/>
+        <child link="camera_link_optical"/>
+        <origin xyz="0 0 0" rpy="${-pi/2} 0 ${-pi/2}"/>
+  </joint>
+  <link name="camera_link_optical"></link>
 </robot>
